File: files/PSprogramboard.brd (EAGLE design)
At the start: 61.9 x 64.8 mm, 13 parts, among them X1 22-23-2021

Commit message: polycutter
Parts:
- moved JP2 38.9 mm to (57.1, 57.1)
- moved U$1 30.1 mm to (38.7, 29.2), turned to 90 degrees
- moved JP3 26.2 mm to (57.1, 41.9)
- moved R1 23.9 mm to (43.8, 29.2), turned to 270 degrees
- moved JP4 15.4 mm to (57.1, 49.5), turned to 0 degrees
- moved X1 0.63 mm to (19.1, 14.6)
Connections:
- removed net N$5 (its old number): JP1.9, JP3.4
- removed net N$7 (its old number): JP2.4, LENGHT1.4
- new net N$10: JP2.4, LENGHT1.2
- new net N$2: JP1.10, JP3.1
- net N$1: now also LENGHT1.5; no longer LENGHT1.1
- net N$12: now also LENGHT1.1; no longer LENGHT1.5
- net N$13: now also JP3.5; no longer JP3.1
- net N$4: now also JP1.9, JP3.2; no longer JP1.10, JP3.5
- net N$6: now also LENGHT1.4; no longer LENGHT1.2
- net N$8: now also JP3.4; no longer JP3.2
Routing:
- net GND: track 164.9 -> 48.3 mm
- net N$10: track 0.00 -> 57.7 mm
- net N$12: track 7.62 -> 64.8 mm
- net N$13: track 6.35 -> 51.5 mm
- net N$7: track 7.62 -> 49.4 mm
- net N$8: track 6.35 -> 45.0 mm
- net VCC: track 172.7 -> 137.0 mm
- net N$6: track 7.62 -> 41.6 mm
- net N$5: track 6.35 -> 37.4 mm
- net N$1: track 7.62 -> 35.1 mm
- net N$4: track 6.35 -> 29.4 mm
- net N$2: track 0.00 -> 22.1 mm
- net N$18: track 13.0 -> 31.3 mm
- net N$17: track 16.6 -> 26.8 mm
- net N$7 (its old number): track 7.62 -> 0.00 mm
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Other:
- board size 61.9 x 64.8 mm -> 64.4 x 64.8 mm
